Commit message: [hui_hardware] align all file & [real] add effort checking

File: rsc/ur5_allegro/ur5_allegro_low_effort.urdf (robot description, URDF)
Before this commit: robot ur5, 35 links, 34 joints
Joints:
- joint joint_0.0: limit lower=-0.47 upper=0.47 effort=15 velocity=7 -> lower=-0.47 upper=0.47 effort=0.7 velocity=7
- joint joint_1.0: limit lower=-0.196 upper=1.61 effort=15 velocity=7 -> lower=-0.196 upper=1.61 effort=0.7 velocity=7
- joint joint_10.0: limit lower=-0.174 upper=1.709 effort=15 velocity=7 -> lower=-0.174 upper=1.709 effort=0.7 velocity=7
- joint joint_11.0: limit lower=-0.227 upper=1.618 effort=15 velocity=7 -> lower=-0.227 upper=1.618 effort=0.7 velocity=7
- joint joint_12.0: limit lower=0.263 upper=1.396 effort=15 velocity=7 -> lower=0.263 upper=1.396 effort=0.7 velocity=7
- joint joint_13.0: limit lower=-0.105 upper=1.163 effort=15 velocity=7 -> lower=-0.105 upper=1.163 effort=0.7 velocity=7
- joint joint_14.0: limit lower=-0.189 upper=1.644 effort=15 velocity=7 -> lower=-0.189 upper=1.644 effort=0.7 velocity=7
- joint joint_15.0: limit lower=-0.162 upper=1.719 effort=15 velocity=7 -> lower=-0.162 upper=1.719 effort=0.7 velocity=7
- joint joint_2.0: limit lower=-0.174 upper=1.709 effort=15 velocity=7 -> lower=-0.174 upper=1.709 effort=0.7 velocity=7
- joint joint_3.0: limit lower=-0.227 upper=1.618 effort=15 velocity=7 -> lower=-0.227 upper=1.618 effort=0.7 velocity=7
- joint joint_4.0: limit lower=-0.47 upper=0.47 effort=15 velocity=7 -> lower=-0.47 upper=0.47 effort=0.7 velocity=7
- joint joint_5.0: limit lower=-0.196 upper=1.61 effort=15 velocity=7 -> lower=-0.196 upper=1.61 effort=0.7 velocity=7
- joint joint_6.0: limit lower=-0.174 upper=1.709 effort=15 velocity=7 -> lower=-0.174 upper=1.709 effort=0.7 velocity=7
- joint joint_7.0: limit lower=-0.227 upper=1.618 effort=15 velocity=7 -> lower=-0.227 upper=1.618 effort=0.7 velocity=7
- joint joint_8.0: limit lower=-0.47 upper=0.47 effort=15 velocity=7 -> lower=-0.47 upper=0.47 effort=0.7 velocity=7
- joint joint_9.0: limit lower=-0.196 upper=1.61 effort=15 velocity=7 -> lower=-0.196 upper=1.61 effort=0.7 velocity=7

File: rsc/ur5_allegro/ur5_allegro_low_effort_mass.urdf (robot description, URDF)
Before this commit: robot ur5, 35 links, 34 joints
Links:
- link link_0.0: mass 0.0119 -> 0.01458
- link link_1.0: mass 0.065 -> 0.0796
- link link_10.0: mass 0.0355 -> 0.04349
- link link_11.0: mass 0.0096 -> 0.01103
- link link_11.0_tip: mass 0.0168 -> 0.02058
- link link_12.0: mass 0.0176 -> 0.0272
- link link_13.0: mass 0.0119 -> 0.01836
- link link_14.0: mass 0.038 -> 0.05863
- link link_15.0: mass 0.0388 -> 0.05987
- link link_15.0_tip: mass 0.0168 -> 0.0259224
- link link_2.0: mass 0.0355 -> 0.04349
- link link_3.0: mass 0.0096 -> 0.01103
- link link_3.0_tip: mass 0.0168 -> 0.02058
- link link_4.0: mass 0.0119 -> 0.01458
- link link_5.0: mass 0.065 -> 0.0796
- link link_6.0: mass 0.0355 -> 0.04349
- link link_7.0: mass 0.0096 -> 0.01103
- link link_7.0_tip: mass 0.0168 -> 0.02058
- link link_8.0: mass 0.0119 -> 0.01458
- link link_9.0: mass 0.065 -> 0.0796
Joints:
- joint joint_0.0: limit lower=-0.47 upper=0.47 effort=15 velocity=7 -> lower=-0.47 upper=0.47 effort=0.7 velocity=7
- joint joint_1.0: limit lower=-0.196 upper=1.61 effort=15 velocity=7 -> lower=-0.196 upper=1.61 effort=0.7 velocity=7
- joint joint_10.0: limit lower=-0.174 upper=1.709 effort=15 velocity=7 -> lower=-0.174 upper=1.709 effort=0.7 velocity=7
- joint joint_11.0: limit lower=-0.227 upper=1.618 effort=15 velocity=7 -> lower=-0.227 upper=1.618 effort=0.7 velocity=7
- joint joint_12.0: limit lower=0.263 upper=1.396 effort=15 velocity=7 -> lower=0.263 upper=1.396 effort=0.7 velocity=7
- joint joint_13.0: limit lower=-0.105 upper=1.163 effort=15 velocity=7 -> lower=-0.105 upper=1.163 effort=0.7 velocity=7
- joint joint_14.0: limit lower=-0.189 upper=1.644 effort=15 velocity=7 -> lower=-0.189 upper=1.644 effort=0.7 velocity=7
- joint joint_15.0: limit lower=-0.162 upper=1.719 effort=15 velocity=7 -> lower=-0.162 upper=1.719 effort=0.7 velocity=7
- joint joint_2.0: limit lower=-0.174 upper=1.709 effort=15 velocity=7 -> lower=-0.174 upper=1.709 effort=0.7 velocity=7
- joint joint_3.0: limit lower=-0.227 upper=1.618 effort=15 velocity=7 -> lower=-0.227 upper=1.618 effort=0.7 velocity=7
- joint joint_4.0: limit lower=-0.47 upper=0.47 effort=15 velocity=7 -> lower=-0.47 upper=0.47 effort=0.7 velocity=7
- joint joint_5.0: limit lower=-0.196 upper=1.61 effort=15 velocity=7 -> lower=-0.196 upper=1.61 effort=0.7 velocity=7
- joint joint_6.0: limit lower=-0.174 upper=1.709 effort=15 velocity=7 -> lower=-0.174 upper=1.709 effort=0.7 velocity=7
- joint joint_7.0: limit lower=-0.227 upper=1.618 effort=15 velocity=7 -> lower=-0.227 upper=1.618 effort=0.7 velocity=7
- joint joint_8.0: limit lower=-0.47 upper=0.47 effort=15 velocity=7 -> lower=-0.47 upper=0.47 effort=0.7 velocity=7
- joint joint_9.0: limit lower=-0.196 upper=1.61 effort=15 velocity=7 -> lower=-0.196 upper=1.61 effort=0.7 velocity=7

File: rsc/ur5_allegro/ur5_allegro_ori_coll.urdf (robot description, URDF)
Before this commit: robot ur5, 35 links, 34 joints
Links:
- link Allegro_base_link: geometry collision box size=0.0408 0.1130 0.095; visual mesh filename=allegro_meshes/base_link.STL
- link link_0.0: geometry collision box size=0.0196 0.0275 0.0164; visual mesh filename=allegro_meshes/link_0.0.STL
- link link_1.0: geometry collision box size=0.0196 0.0275 0.054; visual mesh filename=allegro_meshes/link_1.0.STL
- link link_10.0: geometry collision box size=0.0196 0.0275 0.0384; visual mesh filename=allegro_meshes/link_2.0.STL
- link link_11.0: geometry collision box size=0.0196 0.0275 0.0267; visual mesh filename=allegro_meshes/link_3.0.STL
- link link_11.0_tip: geometry collision sphere radius=0.012; visual mesh filename=allegro_meshes/link_3.0_tip.STL
- link link_12.0: geometry collision box size=0.0358 0.034 0.0455; visual mesh filename=allegro_meshes/link_12.0_right.STL
- link link_13.0: geometry collision box size=0.0196 0.0275 0.0177; visual mesh filename=allegro_meshes/link_13.0.STL
- link link_14.0: geometry collision box size=0.0196 0.0275 0.0514; visual mesh filename=allegro_meshes/link_14.0.STL
- link link_15.0: geometry collision box size=0.0196 0.0275 0.0423; visual mesh filename=allegro_meshes/link_15.0.STL
- link link_15.0_tip: geometry collision sphere radius=0.012; visual mesh filename=allegro_meshes/link_15.0_tip.STL
- link link_2.0: geometry collision box size=0.0196 0.0275 0.0384; visual mesh filename=allegro_meshes/link_2.0.STL
- link link_3.0: geometry collision box size=0.0196 0.0275 0.0267; visual mesh filename=allegro_meshes/link_3.0.STL
- link link_3.0_tip: geometry collision sphere radius=0.012; visual mesh filename=allegro_meshes/link_3.0_tip.STL
- link link_4.0: geometry collision box size=0.0196 0.0275 0.0164; visual mesh filename=allegro_meshes/link_0.0.STL
- link link_5.0: geometry collision box size=0.0196 0.0275 0.054; visual mesh filename=allegro_meshes/link_1.0.STL
- link link_6.0: geometry collision box size=0.0196 0.0275 0.0384; visual mesh filename=allegro_meshes/link_2.0.STL
- link link_7.0: geometry collision box size=0.0196 0.0275 0.0267; visual mesh filename=allegro_meshes/link_3.0.STL
- link link_7.0_tip: geometry collision sphere radius=0.012; visual mesh filename=allegro_meshes/link_3.0_tip.STL
- link link_8.0: geometry collision box size=0.0196 0.0275 0.0164; visual mesh filename=allegro_meshes/link_0.0.STL
- link link_9.0: geometry collision box size=0.0196 0.0275 0.054; visual mesh filename=allegro_meshes/link_1.0.STL

File: rsc/ur5_allegro/ur5_allegro_ori_low_effort_mass_new_damping.urdf (robot description, URDF)
Before this commit: robot ur5, 35 links, 34 joints
Links:
- link link_0.0: mass 0.0119 -> 0.01458
- link link_1.0: mass 0.065 -> 0.0796
- link link_10.0: mass 0.0355 -> 0.04349
- link link_11.0: mass 0.0096 -> 0.01103
- link link_11.0_tip: mass 0.0168 -> 0.02058
- link link_12.0: mass 0.0176 -> 0.0272
- link link_13.0: mass 0.0119 -> 0.01836
- link link_14.0: mass 0.038 -> 0.05863
- link link_15.0: mass 0.0388 -> 0.05987
- link link_15.0_tip: mass 0.0168 -> 0.0259224
- link link_2.0: mass 0.0355 -> 0.04349
- link link_3.0: mass 0.0096 -> 0.01103
- link link_3.0_tip: mass 0.0168 -> 0.02058
- link link_4.0: mass 0.0119 -> 0.01458
- link link_5.0: mass 0.065 -> 0.0796
- link link_6.0: mass 0.0355 -> 0.04349
- link link_7.0: mass 0.0096 -> 0.01103
- link link_7.0_tip: mass 0.0168 -> 0.02058
- link link_8.0: mass 0.0119 -> 0.01458
- link link_9.0: mass 0.065 -> 0.0796
Joints:
- joint joint_0.0: limit lower=-0.47 upper=0.47 effort=15 velocity=7 -> lower=-0.47 upper=0.47 effort=0.7 velocity=7
- joint joint_1.0: limit lower=-0.196 upper=1.61 effort=15 velocity=7 -> lower=-0.196 upper=1.61 effort=0.7 velocity=7
- joint joint_10.0: limit lower=-0.174 upper=1.709 effort=15 velocity=7 -> lower=-0.174 upper=1.709 effort=0.7 velocity=7
- joint joint_11.0: limit lower=-0.227 upper=1.618 effort=15 velocity=7 -> lower=-0.227 upper=1.618 effort=0.7 velocity=7
- joint joint_12.0: limit lower=0.263 upper=1.396 effort=15 velocity=7 -> lower=0.263 upper=1.396 effort=0.7 velocity=7
- joint joint_13.0: limit lower=-0.105 upper=1.163 effort=15 velocity=7 -> lower=-0.105 upper=1.163 effort=0.7 velocity=7
- joint joint_14.0: limit lower=-0.189 upper=1.644 effort=15 velocity=7 -> lower=-0.189 upper=1.644 effort=0.7 velocity=7
- joint joint_15.0: limit lower=-0.162 upper=1.719 effort=15 velocity=7 -> lower=-0.162 upper=1.719 effort=0.7 velocity=7
- joint joint_2.0: limit lower=-0.174 upper=1.709 effort=15 velocity=7 -> lower=-0.174 upper=1.709 effort=0.7 velocity=7
- joint joint_3.0: limit lower=-0.227 upper=1.618 effort=15 velocity=7 -> lower=-0.227 upper=1.618 effort=0.7 velocity=7
- joint joint_4.0: limit lower=-0.47 upper=0.47 effort=15 velocity=7 -> lower=-0.47 upper=0.47 effort=0.7 velocity=7
- joint joint_5.0: limit lower=-0.196 upper=1.61 effort=15 velocity=7 -> lower=-0.196 upper=1.61 effort=0.7 velocity=7
- joint joint_6.0: limit lower=-0.174 upper=1.709 effort=15 velocity=7 -> lower=-0.174 upper=1.709 effort=0.7 velocity=7
- joint joint_7.0: limit lower=-0.227 upper=1.618 effort=15 velocity=7 -> lower=-0.227 upper=1.618 effort=0.7 velocity=7
- joint joint_8.0: limit lower=-0.47 upper=0.47 effort=15 velocity=7 -> lower=-0.47 upper=0.47 effort=0.7 velocity=7
- joint joint_9.0: limit lower=-0.196 upper=1.61 effort=15 velocity=7 -> lower=-0.196 upper=1.61 effort=0.7 velocity=7
