Commit message: support left leap hand

File: rsc/ur5_leaphand/ur5_leaphand_fk.urdf (robot description, URDF)
Before this commit: robot ur5, 34 links, 33 joints
Links:
- added link tool0_tmp
Joints:
- added joint Flange2hand_fixed_joint: type fixed, parent tool0_tmp, child tool0, origin xyz=0 0 0 rpy=0 0 0
- joint ee_fixed_joint: origin xyz=0.0 0.0823 0.0 rpy=0.0 0.0 1.57079632679 -> xyz=0.0 0.02 0.0 rpy=0.0 0.0 1.57079632679
- joint wrist_3_link-tool0_fixed_joint: child tool0 -> tool0_tmp; origin xyz=0 0.0823 0 rpy=-1.57079632679 0 0 -> xyz=0 0.05 0 rpy=-1.57079632679 0 0

File: rsc/ur5_leaphand/ur5_leaphand_left.urdf (robot description, URDF)
Before this commit: robot ur5, 35 links, 34 joints
Links:
- removed link palm_lower
- added link palm_lower_left, mass 0.235; collision mesh filename=leap_left_meshes/palm_lower_left.obj; visual mesh filename=leap_left_meshes/palm_lower_left.stl
- link dip: geometry collision mesh filename=leap_left_meshes/dip.obj; visual mesh filename=leap_left_meshes/dip.stl
- link dip_2: geometry collision mesh filename=leap_left_meshes/dip.obj; visual mesh filename=leap_left_meshes/dip.stl
- link dip_3: geometry collision mesh filename=leap_left_meshes/dip.obj; visual mesh filename=leap_left_meshes/dip.stl
- link fingertip: geometry collision mesh filename=leap_left_meshes/fingertip.obj; visual mesh filename=leap_left_meshes/fingertip.stl
- link fingertip_2: geometry collision mesh filename=leap_left_meshes/fingertip.obj; visual mesh filename=leap_left_meshes/fingertip.stl
- link fingertip_3: geometry collision mesh filename=leap_left_meshes/fingertip.obj; visual mesh filename=leap_left_meshes/fingertip.stl
- link mcp_joint: geometry collision mesh filename=leap_left_meshes/mcp_joint.obj; visual mesh filename=leap_left_meshes/mcp_joint.stl
- link mcp_joint_2: geometry collision mesh filename=leap_left_meshes/mcp_joint.obj; visual mesh filename=leap_left_meshes/mcp_joint.stl
- link mcp_joint_3: geometry collision mesh filename=leap_left_meshes/mcp_joint.obj; visual mesh filename=leap_left_meshes/mcp_joint.stl
- link pip: geometry collision mesh filename=leap_left_meshes/pip.obj; visual mesh filename=leap_left_meshes/pip.stl
- link pip_2: geometry collision mesh filename=leap_left_meshes/pip.obj; visual mesh filename=leap_left_meshes/pip.stl
- link pip_3: geometry collision mesh filename=leap_left_meshes/pip.obj; visual mesh filename=leap_left_meshes/pip.stl
- link pip_4: geometry collision mesh filename=leap_left_meshes/pip.obj; visual mesh filename=leap_left_meshes/pip.stl
- link thumb_dip: geometry collision mesh filename=leap_left_meshes/thumb_dip.obj; visual mesh filename=leap_left_meshes/thumb_dip.stl
- link thumb_fingertip: geometry collision mesh filename=leap_left_meshes/thumb_fingertip.obj; visual mesh filename=leap_left_meshes/thumb_fingertip.stl
- link thumb_pip: geometry collision mesh filename=leap_left_meshes/thumb_pip.obj; visual mesh filename=leap_left_meshes/thumb_pip.stl
Joints:
- joint leap_joint0: origin xyz=-0.012200000000000007713 0.038099999999999994982 -0.0025 rpy=-1.570796326794896558 -1.0065212660796336576e-15 1.5707963267948943376 -> xyz=-0.012200000000000005979 0.038100000000000001921 0.014499999999999985123 rpy=-1.57079632679489678 2.8029314871654157891e-15 1.570796326794896336
- joint leap_joint1: origin xyz=-0.0070952496528625457958 0.006057756134899472233 -0.01872240357846021927 rpy=1.5707963267948950037 1.5707963267948945596 0 -> xyz=-0.082574224938392518092 -0.085740011501137525229 0.0078008885838987494094 rpy=1.5707963267948987784 1.570796326794896558 0; parent palm_lower -> palm_lower_left
- joint leap_joint10: origin xyz=0.014999999999999971689 -0.0027 -0.012999999999999959505 rpy=1.5707963267948958919 -1.570796326794896336 0 -> xyz=0.01499999999999996822 0.014299999999999989803 -0.013000000000000025424 rpy=1.5707963267948958919 -1.570796326794896336 0
- joint leap_joint11: origin xyz=9.7144514654701197287e-17 -0.036099999999999868305 0.00020000000000007511769 rpy=4.5935029425113685044e-17 -2.8730071914463799514e-16 1.5565411607615035382e-32 -> xyz=1.0234868508263161857e-16 -0.036099999999999868305 0.00020000000000007858714 rpy=4.5935029425113685044e-17 -2.8730071914463799514e-16 1.5565411607615035382e-32
- joint leap_joint12: limit lower=-0.349 upper=2.094 effort=0.95 velocity=8.48 -> lower=-2.443 upper=0.47 effort=0.95 velocity=8.48; origin xyz=-0.069395249652862533996 -0.0012422438651005258004 -0.021622403578460215601 rpy=-8.2381766464939424156e-17 1.5707963267948956698 0 -> xyz=-0.14487422493839263726 -0.090040011501137440231 0.004900888583899039308 rpy=3.5629789726327258012e-15 1.5707963267948961139 0; parent palm_lower -> palm_lower_left
- joint leap_joint13: limit lower=-0.47 upper=2.443 effort=0.95 velocity=8.48 -> lower=-2.094 upper=0.349 effort=0.95 velocity=8.48; origin xyz=-2.7755575615628913511e-17 0.014300000000000005415 -0.013000000000000011546 rpy=1.5707963267948958919 -1.570796326794896336 0 -> xyz=-1.0148132334464321502e-16 -0.014100000000000126321 -0.012999999999999956035 rpy=-1.570796326794896336 -1.570796326794896336 0
- joint leap_joint14: origin xyz=0 -0.0025 -0.017000000000000053263 rpy=-1.570796326794896558 1.6050198443300131245e-46 -1.9721522630516624601e-31 -> xyz=0 0.014499999999999967776 -0.017000000000000042855 rpy=-1.570796326794896558 -1.5671206742950610653e-15 -5.6898930012051145053e-16
- joint leap_joint15: origin xyz=-1.249000902703301108e-16 0.046599999999999863753 0.00019999999999997710581 rpy=1.5063958491491781023e-44 5.4234187233935260503e-31 3.141592653589793116 -> xyz=-1.1102230246251565404e-16 0.046599999999999683342 0.00020000000000065451533 rpy=-3.1092019091748562186e-17 -4.9644253794601335075e-16 -3.1415926535897846783
- joint leap_joint2: origin xyz=0.01499999999999996822 -0.0027 -0.012999999999999824196 rpy=1.5707963267948958919 -1.570796326794896336 0 -> xyz=0.014999999999999961281 0.014299999999999993272 -0.013000000000000025424 rpy=1.5707963267948958919 -1.570796326794896336 0
- joint leap_joint3: origin xyz=-4.0880582495572692636e-09 -0.036100004210367367397 0.00020000000000007858714 rpy=4.5935029425113685044e-17 -2.8730071914463794583e-16 4.4395481053923607589e-32 -> xyz=-4.0880582469551840497e-09 -0.03610000421036734658 0.0002000000000000612399 rpy=4.5935029425113685044e-17 -2.8730071914463794583e-16 4.4395481053923607589e-32
- joint leap_joint4: origin xyz=-0.012200000000000019856 0.038099999999999981104 -0.0025 rpy=-1.570796326794896558 -1.0065212760057939085e-15 1.5707963267948943376 -> xyz=-0.012200000000000002509 0.038099999999999988043 0.014499999999999999001 rpy=-1.570796326794896558 1.6094417208041279902e-15 1.5707963267948943376
- joint leap_joint5: origin xyz=-0.0070952496528625388569 -0.039392243865100525113 -0.018722403578460229678 rpy=1.570796326794896558 1.570796326794896558 0 -> xyz=-0.08257422493900856697 -0.040290011501137479311 0.007800888583679612201 rpy=1.5707963267948992225 1.570796326794896558 0; parent palm_lower -> palm_lower_left
- joint leap_joint6: origin xyz=0.014999999999999975159 -0.0027 -0.013000000000000018485 rpy=1.5707963267948958919 -1.570796326794896336 0 -> xyz=0.01499999999999996475 0.014299999999999986333 -0.013000000000000025424 rpy=1.5707963267948958919 -1.570796326794896336 0
- joint leap_joint7: origin xyz=1.0061396160665481148e-16 -0.036099999999999854428 0.00020000000000007858714 rpy=4.5935029425113654229e-17 -2.8730071914463794583e-16 1.4408183216511868558e-31 -> xyz=1.0408340855860842566e-16 -0.036099999999999875244 0.00020000000000007511769 rpy=4.5935029425113654229e-17 -2.8730071914463794583e-16 1.4408183216511868558e-31
- joint leap_joint8: origin xyz=-0.012200000000000004244 0.038100000000000001921 -0.0025 rpy=-1.570796326794896558 -1.0065212660796360242e-15 1.5707963267948943376 -> xyz=-0.012200000000000002509 0.038100000000000001921 0.01450000000000000247 rpy=-1.57079632679489678 2.8029314871654240721e-15 1.570796326794896336
- joint leap_joint9: origin xyz=-0.0070952454426398371343 -0.084842243865100515521 -0.018722407666402932774 rpy=1.5707963267948950037 1.5707963267948945596 0 -> xyz=-0.082574224938392323803 0.0051599884988625839555 0.0078008885838987598177 rpy=1.5707963267948987784 1.570796326794896558 0; parent palm_lower -> palm_lower_left
- joint tool0-leaphand_fixed_joint: child palm_lower -> palm_lower_left
- joint wrist_3_link-tool0_fixed_joint: origin xyz=0 0.05 0 rpy=-1.57079632679 0 0 -> xyz=0.075 0.078 0.02 rpy=-1.57079632679 0 0

File: rsc/ur5_leaphand/ur5_leaphand_left_fk.urdf (robot description, URDF)
Before this commit: robot ur5, 35 links, 34 joints
Links:
- removed link palm_lower
- added link palm_lower_left, mass 0.235; collision mesh filename=leap_left_meshes/palm_lower_left.obj; visual mesh filename=leap_left_meshes/palm_lower_left.stl
- link dip: geometry collision mesh filename=leap_left_meshes/dip.obj; visual mesh filename=leap_left_meshes/dip.stl
- link dip_2: geometry collision mesh filename=leap_left_meshes/dip.obj; visual mesh filename=leap_left_meshes/dip.stl
- link dip_3: geometry collision mesh filename=leap_left_meshes/dip.obj; visual mesh filename=leap_left_meshes/dip.stl
- link fingertip: geometry collision mesh filename=leap_left_meshes/fingertip.obj; visual mesh filename=leap_left_meshes/fingertip.stl
- link fingertip_2: geometry collision mesh filename=leap_left_meshes/fingertip.obj; visual mesh filename=leap_left_meshes/fingertip.stl
- link fingertip_3: geometry collision mesh filename=leap_left_meshes/fingertip.obj; visual mesh filename=leap_left_meshes/fingertip.stl
- link mcp_joint: geometry collision mesh filename=leap_left_meshes/mcp_joint.obj; visual mesh filename=leap_left_meshes/mcp_joint.stl
- link mcp_joint_2: geometry collision mesh filename=leap_left_meshes/mcp_joint.obj; visual mesh filename=leap_left_meshes/mcp_joint.stl
- link mcp_joint_3: geometry collision mesh filename=leap_left_meshes/mcp_joint.obj; visual mesh filename=leap_left_meshes/mcp_joint.stl
- link pip: geometry collision mesh filename=leap_left_meshes/pip.obj; visual mesh filename=leap_left_meshes/pip.stl
- link pip_2: geometry collision mesh filename=leap_left_meshes/pip.obj; visual mesh filename=leap_left_meshes/pip.stl
- link pip_3: geometry collision mesh filename=leap_left_meshes/pip.obj; visual mesh filename=leap_left_meshes/pip.stl
- link pip_4: geometry collision mesh filename=leap_left_meshes/pip.obj; visual mesh filename=leap_left_meshes/pip.stl
- link thumb_dip: geometry collision mesh filename=leap_left_meshes/thumb_dip.obj; visual mesh filename=leap_left_meshes/thumb_dip.stl
- link thumb_fingertip: geometry collision mesh filename=leap_left_meshes/thumb_fingertip.obj; visual mesh filename=leap_left_meshes/thumb_fingertip.stl
- link thumb_pip: geometry collision mesh filename=leap_left_meshes/thumb_pip.obj; visual mesh filename=leap_left_meshes/thumb_pip.stl
Joints:
- joint leap_joint0: origin xyz=-0.012200000000000007713 0.038099999999999994982 -0.0025 rpy=-1.570796326794896558 -1.0065212660796336576e-15 1.5707963267948943376 -> xyz=-0.012200000000000005979 0.038100000000000001921 0.014499999999999985123 rpy=-1.57079632679489678 2.8029314871654157891e-15 1.570796326794896336
- joint leap_joint1: origin xyz=-0.0070952496528625457958 0.006057756134899472233 -0.01872240357846021927 rpy=1.5707963267948950037 1.5707963267948945596 0 -> xyz=-0.082574224938392518092 -0.085740011501137525229 0.0078008885838987494094 rpy=1.5707963267948987784 1.570796326794896558 0; parent palm_lower -> palm_lower_left
- joint leap_joint10: origin xyz=0.014999999999999971689 -0.0027 -0.012999999999999959505 rpy=1.5707963267948958919 -1.570796326794896336 0 -> xyz=0.01499999999999996822 0.014299999999999989803 -0.013000000000000025424 rpy=1.5707963267948958919 -1.570796326794896336 0
- joint leap_joint11: origin xyz=9.7144514654701197287e-17 -0.036099999999999868305 0.00020000000000007511769 rpy=4.5935029425113685044e-17 -2.8730071914463799514e-16 1.5565411607615035382e-32 -> xyz=1.0234868508263161857e-16 -0.036099999999999868305 0.00020000000000007858714 rpy=4.5935029425113685044e-17 -2.8730071914463799514e-16 1.5565411607615035382e-32
- joint leap_joint12: limit lower=-0.349 upper=2.094 effort=0.95 velocity=8.48 -> lower=-2.443 upper=0.47 effort=0.95 velocity=8.48; origin xyz=-0.069395249652862533996 -0.0012422438651005258004 -0.021622403578460215601 rpy=-8.2381766464939424156e-17 1.5707963267948956698 0 -> xyz=-0.14487422493839263726 -0.090040011501137440231 0.004900888583899039308 rpy=3.5629789726327258012e-15 1.5707963267948961139 0; parent palm_lower -> palm_lower_left
- joint leap_joint13: limit lower=-0.47 upper=2.443 effort=0.95 velocity=8.48 -> lower=-2.094 upper=0.349 effort=0.95 velocity=8.48; origin xyz=-2.7755575615628913511e-17 0.014300000000000005415 -0.013000000000000011546 rpy=1.5707963267948958919 -1.570796326794896336 0 -> xyz=-1.0148132334464321502e-16 -0.014100000000000126321 -0.012999999999999956035 rpy=-1.570796326794896336 -1.570796326794896336 0
- joint leap_joint14: origin xyz=0 -0.0025 -0.017000000000000053263 rpy=-1.570796326794896558 1.6050198443300131245e-46 -1.9721522630516624601e-31 -> xyz=0 0.014499999999999967776 -0.017000000000000042855 rpy=-1.570796326794896558 -1.5671206742950610653e-15 -5.6898930012051145053e-16
- joint leap_joint15: origin xyz=-1.249000902703301108e-16 0.046599999999999863753 0.00019999999999997710581 rpy=1.5063958491491781023e-44 5.4234187233935260503e-31 3.141592653589793116 -> xyz=-1.1102230246251565404e-16 0.046599999999999683342 0.00020000000000065451533 rpy=-3.1092019091748562186e-17 -4.9644253794601335075e-16 -3.1415926535897846783
- joint leap_joint2: origin xyz=0.01499999999999996822 -0.0027 -0.012999999999999824196 rpy=1.5707963267948958919 -1.570796326794896336 0 -> xyz=0.014999999999999961281 0.014299999999999993272 -0.013000000000000025424 rpy=1.5707963267948958919 -1.570796326794896336 0
- joint leap_joint3: origin xyz=-4.0880582495572692636e-09 -0.036100004210367367397 0.00020000000000007858714 rpy=4.5935029425113685044e-17 -2.8730071914463794583e-16 4.4395481053923607589e-32 -> xyz=-4.0880582469551840497e-09 -0.03610000421036734658 0.0002000000000000612399 rpy=4.5935029425113685044e-17 -2.8730071914463794583e-16 4.4395481053923607589e-32
- joint leap_joint4: origin xyz=-0.012200000000000019856 0.038099999999999981104 -0.0025 rpy=-1.570796326794896558 -1.0065212760057939085e-15 1.5707963267948943376 -> xyz=-0.012200000000000002509 0.038099999999999988043 0.014499999999999999001 rpy=-1.570796326794896558 1.6094417208041279902e-15 1.5707963267948943376
- joint leap_joint5: origin xyz=-0.0070952496528625388569 -0.039392243865100525113 -0.018722403578460229678 rpy=1.570796326794896558 1.570796326794896558 0 -> xyz=-0.08257422493900856697 -0.040290011501137479311 0.007800888583679612201 rpy=1.5707963267948992225 1.570796326794896558 0; parent palm_lower -> palm_lower_left
- joint leap_joint6: origin xyz=0.014999999999999975159 -0.0027 -0.013000000000000018485 rpy=1.5707963267948958919 -1.570796326794896336 0 -> xyz=0.01499999999999996475 0.014299999999999986333 -0.013000000000000025424 rpy=1.5707963267948958919 -1.570796326794896336 0
- joint leap_joint7: origin xyz=1.0061396160665481148e-16 -0.036099999999999854428 0.00020000000000007858714 rpy=4.5935029425113654229e-17 -2.8730071914463794583e-16 1.4408183216511868558e-31 -> xyz=1.0408340855860842566e-16 -0.036099999999999875244 0.00020000000000007511769 rpy=4.5935029425113654229e-17 -2.8730071914463794583e-16 1.4408183216511868558e-31
- joint leap_joint8: origin xyz=-0.012200000000000004244 0.038100000000000001921 -0.0025 rpy=-1.570796326794896558 -1.0065212660796360242e-15 1.5707963267948943376 -> xyz=-0.012200000000000002509 0.038100000000000001921 0.01450000000000000247 rpy=-1.57079632679489678 2.8029314871654240721e-15 1.570796326794896336
- joint leap_joint9: origin xyz=-0.0070952454426398371343 -0.084842243865100515521 -0.018722407666402932774 rpy=1.5707963267948950037 1.5707963267948945596 0 -> xyz=-0.082574224938392323803 0.0051599884988625839555 0.0078008885838987598177 rpy=1.5707963267948987784 1.570796326794896558 0; parent palm_lower -> palm_lower_left
- joint tool0-leaphand_fixed_joint: child palm_lower -> palm_lower_left
- joint wrist_3_link-tool0_fixed_joint: origin xyz=0 0.05 0 rpy=-1.57079632679 0 0 -> xyz=0.075 0.078 0.02 rpy=-1.57079632679 0 0
