Commit message: refine the collision body of leaphand

File: rsc/ur5_leaphand/ur5_leaphand.urdf (robot description, URDF)
Before this commit: robot ur5, 35 links, 34 joints
Links:
- link dip: geometry collision box size=0.032 0.018 0.022; visual mesh filename=leap_right_meshes/dip.stl
- link dip_2: geometry collision box size=0.032 0.018 0.022; visual mesh filename=leap_right_meshes/dip.stl
- link dip_3: geometry collision box size=0.032 0.018 0.022; visual mesh filename=leap_right_meshes/dip.stl
- link fingertip: geometry collision mesh filename=leap_right_meshes/fingertip_simplify.obj; visual mesh filename=leap_right_meshes/fingertip.stl
- link fingertip_2: geometry collision mesh filename=leap_right_meshes/fingertip_simplify.obj; visual mesh filename=leap_right_meshes/fingertip.stl
- link fingertip_3: geometry collision mesh filename=leap_right_meshes/fingertip_simplify.obj; visual mesh filename=leap_right_meshes/fingertip.stl
- link mcp_joint: geometry collision box size=0.026 0.038 0.023; visual mesh filename=leap_right_meshes/mcp_joint.stl
- link mcp_joint_2: geometry collision box size=0.026 0.038 0.023; visual mesh filename=leap_right_meshes/mcp_joint.stl
- link mcp_joint_3: geometry collision box size=0.026 0.038 0.023; visual mesh filename=leap_right_meshes/mcp_joint.stl
- link palm_lower: geometry collision mesh filename=leap_right_meshes/palm_lower_simplify.obj; visual mesh filename=leap_right_meshes/palm_lower.stl
- link pip: geometry collision box size=0.048 0.028 0.018; visual mesh filename=leap_right_meshes/pip.stl
- link pip_2: geometry collision box size=0.048 0.028 0.018; visual mesh filename=leap_right_meshes/pip.stl
- link pip_3: geometry collision box size=0.048 0.028 0.018; visual mesh filename=leap_right_meshes/pip.stl
- link pip_4: geometry collision box size=0.03 0.02 0.015; visual mesh filename=leap_right_meshes/pip.stl
- link thumb_dip: geometry collision box size=0.02 0.033 0.02; visual mesh filename=leap_right_meshes/thumb_dip.stl
- link thumb_fingertip: geometry collision mesh filename=leap_right_meshes/thumb_fingertip_simplify.obj; visual mesh filename=leap_right_meshes/thumb_fingertip.stl
- link thumb_pip: geometry collision box size=0.002 0.002 0.002; visual mesh filename=leap_right_meshes/thumb_pip.stl

File: rsc/ur5_leaphand/ur5_leaphand_left.urdf (robot description, URDF)
Before this commit: robot ur5, 35 links, 34 joints
Links:
- link dip: geometry collision box size=0.032 0.018 0.022; visual mesh filename=leap_left_meshes/dip.stl
- link dip_2: geometry collision box size=0.032 0.018 0.022; visual mesh filename=leap_left_meshes/dip.stl
- link dip_3: geometry collision box size=0.032 0.018 0.022; visual mesh filename=leap_left_meshes/dip.stl
- link fingertip: geometry collision mesh filename=leap_left_meshes/fingertip_simplify.obj; visual mesh filename=leap_left_meshes/fingertip.stl
- link fingertip_2: geometry collision mesh filename=leap_left_meshes/fingertip_simplify.obj; visual mesh filename=leap_left_meshes/fingertip.stl
- link fingertip_3: geometry collision mesh filename=leap_left_meshes/fingertip_simplify.obj; visual mesh filename=leap_left_meshes/fingertip.stl
- link mcp_joint: geometry collision box size=0.026 0.038 0.023; visual mesh filename=leap_left_meshes/mcp_joint.stl
- link mcp_joint_2: geometry collision box size=0.026 0.038 0.023; visual mesh filename=leap_left_meshes/mcp_joint.stl
- link mcp_joint_3: geometry collision box size=0.026 0.038 0.023; visual mesh filename=leap_left_meshes/mcp_joint.stl
- link palm_lower_left: geometry collision mesh filename=leap_left_meshes/palm_lower_left_simplify.obj; visual mesh filename=leap_left_meshes/palm_lower_left.stl
- link pip: geometry collision box size=0.048 0.028 0.018; visual mesh filename=leap_left_meshes/pip.stl
- link pip_2: geometry collision box size=0.048 0.028 0.018; visual mesh filename=leap_left_meshes/pip.stl
- link pip_3: geometry collision box size=0.048 0.028 0.018; visual mesh filename=leap_left_meshes/pip.stl
- link pip_4: geometry collision box size=0.03 0.02 0.015; visual mesh filename=leap_left_meshes/pip.stl
- link thumb_dip: geometry collision box size=0.02 0.033 0.02; visual mesh filename=leap_left_meshes/thumb_dip.stl
- link thumb_fingertip: geometry collision mesh filename=leap_left_meshes/thumb_fingertip_simplify.obj; visual mesh filename=leap_left_meshes/thumb_fingertip.stl
- link thumb_pip: geometry collision box size=0.002 0.002 0.002; visual mesh filename=leap_left_meshes/thumb_pip.stl

Commit message: update collision body of leaphand

File: rsc/ur5_leaphand/ur5_leaphand.urdf (robot description, URDF)
Before this commit: robot ur5, 35 links, 34 joints
Links:
- removed link tool0_tmp
- added link Flange_base_link
Joints:
- removed joint tool0-leaphand_fixed_joint
- added joint tool02Flange_fixed_joint: type fixed, parent tool0, child Flange_base_link, origin xyz=-0.03 -0.065 0.025 rpy=-3.14159265 0 -1.57079632679
- joint Flange2hand_fixed_joint: child tool0 -> palm_lower; parent tool0_tmp -> Flange_base_link
- joint wrist_3_link-tool0_fixed_joint: child tool0_tmp -> tool0; origin xyz=0 0.05 0 rpy=-1.57079632679 0 0 -> xyz=0 0.0823 0 rpy=-1.57079632679 0 0

File: rsc/ur5_leaphand/ur5_leaphand_fk.urdf (robot description, URDF)
Before this commit: robot ur5, 35 links, 34 joints
Links:
- removed link tool0_tmp
- added link Flange_base_link
- link dip: geometry collision box size=0.032 0.018 0.022; visual mesh filename=leap_right_meshes/dip.stl
- link dip_2: geometry collision box size=0.032 0.018 0.022; visual mesh filename=leap_right_meshes/dip.stl
- link dip_3: geometry collision box size=0.032 0.018 0.022; visual mesh filename=leap_right_meshes/dip.stl
- link fingertip: geometry collision mesh filename=leap_right_meshes/fingertip_simplify.obj; visual mesh filename=leap_right_meshes/fingertip.stl
- link fingertip_2: geometry collision mesh filename=leap_right_meshes/fingertip_simplify.obj; visual mesh filename=leap_right_meshes/fingertip.stl
- link fingertip_3: geometry collision mesh filename=leap_right_meshes/fingertip_simplify.obj; visual mesh filename=leap_right_meshes/fingertip.stl
- link mcp_joint: geometry collision box size=0.026 0.038 0.023; visual mesh filename=leap_right_meshes/mcp_joint.stl
- link mcp_joint_2: geometry collision box size=0.026 0.038 0.023; visual mesh filename=leap_right_meshes/mcp_joint.stl
- link mcp_joint_3: geometry collision box size=0.026 0.038 0.023; visual mesh filename=leap_right_meshes/mcp_joint.stl
- link palm_lower: geometry collision mesh filename=leap_right_meshes/palm_lower_simplify.obj; visual mesh filename=leap_right_meshes/palm_lower.stl
- link pip: geometry collision box size=0.048 0.028 0.018; visual mesh filename=leap_right_meshes/pip.stl
- link pip_2: geometry collision box size=0.048 0.028 0.018; visual mesh filename=leap_right_meshes/pip.stl
- link pip_3: geometry collision box size=0.048 0.028 0.018; visual mesh filename=leap_right_meshes/pip.stl
- link pip_4: geometry collision box size=0.03 0.02 0.015; visual mesh filename=leap_right_meshes/pip.stl
- link thumb_dip: geometry collision box size=0.02 0.033 0.02; visual mesh filename=leap_right_meshes/thumb_dip.stl
- link thumb_fingertip: geometry collision mesh filename=leap_right_meshes/thumb_fingertip_simplify.obj; visual mesh filename=leap_right_meshes/thumb_fingertip.stl
- link thumb_pip: geometry collision box size=0.002 0.002 0.002; visual mesh filename=leap_right_meshes/thumb_pip.stl
Joints:
- removed joint tool0-leaphand_fixed_joint
- added joint tool02Flange_fixed_joint: type fixed, parent tool0, child Flange_base_link, origin xyz=-0.03 -0.065 0.025 rpy=-3.14159265 0 -1.57079632679
- joint Flange2hand_fixed_joint: child tool0 -> palm_lower; parent tool0_tmp -> Flange_base_link
- joint wrist_3_link-tool0_fixed_joint: child tool0_tmp -> tool0; origin xyz=0 0.05 0 rpy=-1.57079632679 0 0 -> xyz=0 0.0823 0 rpy=-1.57079632679 0 0

File: rsc/ur5_leaphand/ur5_leaphand_left.urdf (robot description, URDF)
Before this commit: robot ur5, 35 links, 34 joints
Links:
- removed link tool0_tmp
- added link Flange_base_link
Joints:
- removed joint tool0-leaphand_fixed_joint
- added joint tool02Flange_fixed_joint: type fixed, parent tool0, child Flange_base_link, origin xyz=-0.06 -0.135 0.05 rpy=-3.14159265 0 -1.57079632679
- joint Flange2hand_fixed_joint: child tool0 -> palm_lower_left; parent tool0_tmp -> Flange_base_link
- joint wrist_3_link-tool0_fixed_joint: child tool0_tmp -> tool0; origin xyz=0.075 0.078 0.02 rpy=-1.57079632679 0 0 -> xyz=0 0.0823 0 rpy=-1.57079632679 0 0

File: rsc/ur5_leaphand/ur5_leaphand_left_fk.urdf (robot description, URDF)
Before this commit: robot ur5, 35 links, 34 joints
Links:
- removed link tool0_tmp
- added link Flange_base_link
- link dip: geometry collision box size=0.032 0.018 0.022; visual mesh filename=leap_left_meshes/dip.stl
- link dip_2: geometry collision box size=0.032 0.018 0.022; visual mesh filename=leap_left_meshes/dip.stl
- link dip_3: geometry collision box size=0.032 0.018 0.022; visual mesh filename=leap_left_meshes/dip.stl
- link fingertip: geometry collision mesh filename=leap_left_meshes/fingertip_simplify.obj; visual mesh filename=leap_left_meshes/fingertip.stl
- link fingertip_2: geometry collision mesh filename=leap_left_meshes/fingertip_simplify.obj; visual mesh filename=leap_left_meshes/fingertip.stl
- link fingertip_3: geometry collision mesh filename=leap_left_meshes/fingertip_simplify.obj; visual mesh filename=leap_left_meshes/fingertip.stl
- link mcp_joint: geometry collision box size=0.026 0.038 0.023; visual mesh filename=leap_left_meshes/mcp_joint.stl
- link mcp_joint_2: geometry collision box size=0.026 0.038 0.023; visual mesh filename=leap_left_meshes/mcp_joint.stl
- link mcp_joint_3: geometry collision box size=0.026 0.038 0.023; visual mesh filename=leap_left_meshes/mcp_joint.stl
- link palm_lower_left: geometry collision mesh filename=leap_left_meshes/palm_lower_left_simplify.obj; visual mesh filename=leap_left_meshes/palm_lower_left.stl
- link pip: geometry collision box size=0.048 0.028 0.018; visual mesh filename=leap_left_meshes/pip.stl
- link pip_2: geometry collision box size=0.048 0.028 0.018; visual mesh filename=leap_left_meshes/pip.stl
- link pip_3: geometry collision box size=0.048 0.028 0.018; visual mesh filename=leap_left_meshes/pip.stl
- link pip_4: geometry collision box size=0.03 0.02 0.015; visual mesh filename=leap_left_meshes/pip.stl
- link thumb_dip: geometry collision box size=0.02 0.033 0.02; visual mesh filename=leap_left_meshes/thumb_dip.stl
- link thumb_fingertip: geometry collision mesh filename=leap_left_meshes/thumb_fingertip_simplify.obj; visual mesh filename=leap_left_meshes/thumb_fingertip.stl
- link thumb_pip: geometry collision box size=0.002 0.002 0.002; visual mesh filename=leap_left_meshes/thumb_pip.stl
Joints:
- removed joint tool0-leaphand_fixed_joint
- added joint tool02Flange_fixed_joint: type fixed, parent tool0, child Flange_base_link, origin xyz=-0.06 -0.135 0.05 rpy=-3.14159265 0 -1.57079632679
- joint Flange2hand_fixed_joint: child tool0 -> palm_lower_left; parent tool0_tmp -> Flange_base_link
- joint wrist_3_link-tool0_fixed_joint: child tool0_tmp -> tool0; origin xyz=0.075 0.078 0.02 rpy=-1.57079632679 0 0 -> xyz=0 0.0823 0 rpy=-1.57079632679 0 0

Commit message: update leaphand urdf

File: rsc/ur5_leaphand/ur5_leaphand.urdf (robot description, URDF)
Before this commit: robot ur5, 35 links, 34 joints
Joints:
- joint Flange2hand_fixed_joint: origin xyz=0 0 0 rpy=0 0 0 -> xyz=-0.03 -0.065 0.025 rpy=-3.14159265 0 -1.57079632679
- joint tool02Flange_fixed_joint: origin xyz=-0.03 -0.065 0.025 rpy=-3.14159265 0 -1.57079632679 -> xyz=0 0 0 rpy=0 0 0

File: rsc/ur5_leaphand/ur5_leaphand_fk.urdf (robot description, URDF)
Before this commit: robot ur5, 35 links, 34 joints
Joints:
- joint Flange2hand_fixed_joint: origin xyz=0 0 0 rpy=0 0 0 -> xyz=-0.03 -0.065 0.025 rpy=-3.14159265 0 -1.57079632679
- joint tool02Flange_fixed_joint: origin xyz=-0.03 -0.065 0.025 rpy=-3.14159265 0 -1.57079632679 -> xyz=0 0 0 rpy=0 0 0

File: rsc/ur5_leaphand/ur5_leaphand_left.urdf (robot description, URDF)
Before this commit: robot ur5, 35 links, 34 joints
Joints:
- joint Flange2hand_fixed_joint: origin xyz=0 0 0 rpy=0 0 0 -> xyz=-0.06 -0.135 0.05 rpy=-3.14159265 0 -1.57079632679
- joint tool02Flange_fixed_joint: origin xyz=-0.06 -0.135 0.05 rpy=-3.14159265 0 -1.57079632679 -> xyz=0 0 0 rpy=0 0 0

File: rsc/ur5_leaphand/ur5_leaphand_left_fk.urdf (robot description, URDF)
Before this commit: robot ur5, 35 links, 34 joints
Joints:
- joint Flange2hand_fixed_joint: origin xyz=0 0 0 rpy=0 0 0 -> xyz=-0.06 -0.135 0.05 rpy=-3.14159265 0 -1.57079632679
- joint tool02Flange_fixed_joint: origin xyz=-0.06 -0.135 0.05 rpy=-3.14159265 0 -1.57079632679 -> xyz=0 0 0 rpy=0 0 0

Commit message: add the ros driver of leaphand

File: rsc/ur5_leaphand/ur5_leaphand.urdf (robot description, URDF)
Before this commit: robot ur5, 35 links, 34 joints
Joints:
- joint leap_joint0: limit lower=-1.047 upper=1.047 effort=0.95 velocity=8.48 -> lower=-0.31 upper=0.31 effort=0.95 velocity=8.48
- joint leap_joint4: limit lower=-1.047 upper=1.047 effort=0.95 velocity=8.48 -> lower=-0.31 upper=0.31 effort=0.95 velocity=8.48
- joint leap_joint8: limit lower=-1.047 upper=1.047 effort=0.95 velocity=8.48 -> lower=-0.31 upper=0.31 effort=0.95 velocity=8.48

File: rsc/ur5_leaphand/ur5_leaphand_left.urdf (robot description, URDF)
Before this commit: robot ur5, 35 links, 34 joints
Joints:
- joint leap_joint0: limit lower=-1.047 upper=1.047 effort=0.95 velocity=8.48 -> lower=-0.31 upper=0.31 effort=0.95 velocity=8.48
- joint leap_joint4: limit lower=-1.047 upper=1.047 effort=0.95 velocity=8.48 -> lower=-0.31 upper=0.31 effort=0.95 velocity=8.48
- joint leap_joint8: limit lower=-1.047 upper=1.047 effort=0.95 velocity=8.48 -> lower=-0.31 upper=0.31 effort=0.95 velocity=8.48
