Commit message: update the collision of left leaphand

File: rsc/ur5_leaphand/ur5_leaphand_left.urdf (robot description, URDF)
Before this commit: robot ur5, 35 links, 34 joints
Links:
- link fingertip: geometry collision mesh filename=leap_left_meshes/fingertip_simplify_simplify.obj; visual mesh filename=leap_left_meshes/fingertip.stl
- link fingertip_2: geometry collision mesh filename=leap_left_meshes/fingertip_simplify_simplify.obj; visual mesh filename=leap_left_meshes/fingertip.stl
- link fingertip_3: geometry collision mesh filename=leap_left_meshes/fingertip_simplify_simplify.obj; visual mesh filename=leap_left_meshes/fingertip.stl
- link palm_lower_left: geometry collision mesh filename=leap_left_meshes/palm_lower_left_simplify_simplify.obj; visual mesh filename=leap_left_meshes/palm_lower_left_simplify.obj
- link thumb_fingertip: geometry collision mesh filename=leap_left_meshes/thumb_fingertip_simplify_simplify.obj; visual mesh filename=leap_left_meshes/thumb_fingertip.stl
Joints:
- joint leap_joint0: origin xyz=-0.012200000000000005979 0.038100000000000001921 0.014499999999999985123 rpy=-1.57079632679489678 2.8029314871654157891e-15 1.570796326794896336 -> xyz=-0.012200000000000005979 0.038100000000000001921 0.0 rpy=-1.57079632679489678 2.8029314871654157891e-15 1.570796326794896336
- joint leap_joint1: origin xyz=-0.082574224938392518092 -0.085740011501137525229 0.0078008885838987494094 rpy=1.5707963267948987784 1.570796326794896558 0 -> xyz=-0.082574224938392518092 -0.1 0.0078008885838987494094 rpy=1.5707963267948987784 1.570796326794896558 0
- joint leap_joint10: origin xyz=0.01499999999999996822 0.014299999999999989803 -0.013000000000000025424 rpy=1.5707963267948958919 -1.570796326794896336 0 -> xyz=0.01499999999999996822 0.0 -0.013000000000000025424 rpy=1.5707963267948958919 -1.570796326794896336 0
- joint leap_joint12: limit lower=-2.443 upper=0.47 effort=0.95 velocity=8.48 -> lower=-2.1 upper=0.3 effort=0.95 velocity=8.48; origin xyz=-0.14487422493839263726 -0.090040011501137440231 0.004900888583899039308 rpy=3.5629789726327258012e-15 1.5707963267948961139 0 -> xyz=-0.14487422493839263726 -0.090040011501137440231 0.015 rpy=3.5629789726327258012e-15 1.5707963267948961139 0
- joint leap_joint14: origin xyz=0 0.014499999999999967776 -0.017000000000000042855 rpy=-1.570796326794896558 -1.5671206742950610653e-15 -5.6898930012051145053e-16 -> xyz=0 0 -0.017000000000000042855 rpy=-1.570796326794896558 -1.5671206742950610653e-15 -5.6898930012051145053e-16
- joint leap_joint2: origin xyz=0.014999999999999961281 0.014299999999999993272 -0.013000000000000025424 rpy=1.5707963267948958919 -1.570796326794896336 0 -> xyz=0.014999999999999961281 0.0 -0.013000000000000025424 rpy=1.5707963267948958919 -1.570796326794896336 0
- joint leap_joint4: origin xyz=-0.012200000000000002509 0.038099999999999988043 0.014499999999999999001 rpy=-1.570796326794896558 1.6094417208041279902e-15 1.5707963267948943376 -> xyz=-0.012200000000000002509 0.038099999999999988043 0.0 rpy=-1.570796326794896558 1.6094417208041279902e-15 1.5707963267948943376
- joint leap_joint5: origin xyz=-0.08257422493900856697 -0.040290011501137479311 0.007800888583679612201 rpy=1.5707963267948992225 1.570796326794896558 0 -> xyz=-0.08257422493900856697 -0.055 0.007800888583679612201 rpy=1.5707963267948992225 1.570796326794896558 0
- joint leap_joint6: origin xyz=0.01499999999999996475 0.014299999999999986333 -0.013000000000000025424 rpy=1.5707963267948958919 -1.570796326794896336 0 -> xyz=0.01499999999999996475 0.0 -0.013000000000000025424 rpy=1.5707963267948958919 -1.570796326794896336 0
- joint leap_joint8: origin xyz=-0.012200000000000002509 0.038100000000000001921 0.01450000000000000247 rpy=-1.57079632679489678 2.8029314871654240721e-15 1.570796326794896336 -> xyz=-0.012200000000000002509 0.038100000000000001921 0.0 rpy=-1.57079632679489678 2.8029314871654240721e-15 1.570796326794896336
- joint leap_joint9: origin xyz=-0.082574224938392323803 0.0051599884988625839555 0.0078008885838987598177 rpy=1.5707963267948987784 1.570796326794896558 0 -> xyz=-0.082574224938392323803 -0.01 0.0078008885838987598177 rpy=1.5707963267948987784 1.570796326794896558 0

Commit message: use solidworks to simplify the mesh of left hand

File: rsc/ur5_leaphand/ur5_leaphand_left.urdf (robot description, URDF)
Before this commit: robot ur5, 35 links, 34 joints
Links:
- link fingertip: geometry collision mesh filename=leap_left_meshes/finger_sw_simplify.obj; visual mesh filename=leap_left_meshes/fingertip.stl
- link fingertip_2: geometry collision mesh filename=leap_left_meshes/finger_sw_simplify.obj; visual mesh filename=leap_left_meshes/fingertip.stl
- link fingertip_3: geometry collision mesh filename=leap_left_meshes/finger_sw_simplify.obj; visual mesh filename=leap_left_meshes/fingertip.stl
- link palm_lower_left: geometry collision mesh filename=leap_left_meshes/palam_sw_simplify.obj; visual mesh filename=leap_left_meshes/palm_lower_left_simplify.obj
- link thumb_fingertip: geometry collision mesh filename=leap_left_meshes/thumb_finger_sw_simplify.obj; visual mesh filename=leap_left_meshes/thumb_fingertip.stl
