Commit message: update the mesh of leaphand using solidowrks

File: rsc/ur5_leaphand/ur5_leaphand_left_sw.urdf (robot description, URDF)
Before this commit: robot ur5, 35 links, 34 joints
Links:
- link fingertip: geometry collision mesh filename=leap_left_meshes/tip.obj; visual mesh filename=leap_left_meshes/fingertip.stl
- link fingertip_2: geometry collision mesh filename=leap_left_meshes/tip.obj; visual mesh filename=leap_left_meshes/fingertip.stl
- link fingertip_3: geometry collision mesh filename=leap_left_meshes/tip.obj; visual mesh filename=leap_left_meshes/fingertip.stl
- link palm_lower_left: geometry collision mesh filename=leap_left_meshes/palam_sw.obj; visual mesh filename=leap_left_meshes/palm_lower_left_simplify.obj

File: rsc/ur5_leaphand/ur5_leaphand_right_sw.urdf (robot description, URDF)
Before this commit: robot ur5, 35 links, 34 joints
Links:
- link fingertip: mass 0.016 -> 0.006; geometry collision mesh filename=leap_left_meshes/finger_sw.obj; visual mesh filename=leap_right_meshes/fingertip.stl
- link fingertip_2: mass 0.016 -> 0.006; geometry collision mesh filename=leap_left_meshes/finger_sw.obj; visual mesh filename=leap_right_meshes/fingertip.stl
- link fingertip_3: mass 0.016 -> 0.006; geometry collision mesh filename=leap_left_meshes/finger_sw.obj; visual mesh filename=leap_right_meshes/fingertip.stl
- link leap_link11_tip: mass None -> 0.01; geometry collision mesh filename=leap_left_meshes/tip.obj
- link leap_link15_tip: mass None -> 0.01; geometry collision mesh filename=leap_left_meshes/tip.obj
- link leap_link3_tip: mass None -> 0.01; geometry collision mesh filename=leap_left_meshes/tip.obj
- link leap_link7_tip: mass None -> 0.01; geometry collision mesh filename=leap_left_meshes/tip.obj
- link palm_lower: geometry collision mesh filename=leap_right_meshes/palam_right_sw.obj; visual mesh filename=leap_right_meshes/palm_lower_simplify.obj
- link thumb_fingertip: mass 0.049 -> 0.039; geometry collision box size=0.02 0.04 0.025; visual mesh filename=leap_right_meshes/thumb_fingertip.stl
