Commit message: update the param while training leaphand

File: rsc/ur5_leaphand/ur5_leaphand_left_sw_noinertia.urdf (robot description, URDF)
Before this commit: robot ur5, 35 links, 34 joints
Links:
- link thumb_fingertip: geometry collision mesh filename=leap_left_meshes/thumb_tip_new.obj; visual mesh filename=leap_left_meshes/thumb_fingertip.stl
Joints:
- joint leap_joint12: limit lower=-2.0 upper=0.0 effort=0.95 velocity=8.48 -> lower=-1.9 upper=0. effort=0.95 velocity=8.48
- joint leap_joint13: limit lower=-0.3 upper=0.1 effort=0.95 velocity=8.48 -> lower=-0.3 upper=0.3 effort=0.95 velocity=8.48

Commit message: update the param of traning leaphand

File: rsc/ur5_leaphand/ur5_leaphand_left_sw_noinertia.urdf (robot description, URDF)
Before this commit: robot ur5, 35 links, 34 joints
Joints:
- joint leap_joint12: limit lower=-1.9 upper=0. effort=0.95 velocity=8.48 -> lower=-1.9 upper=0. effort=2.0 velocity=8.48
- joint leap_joint13: limit lower=-0.3 upper=0.3 effort=0.95 velocity=8.48 -> lower=-0.3 upper=0.3 effort=2.0 velocity=8.48
- joint leap_joint14: limit lower=-1.20 upper=1.90 effort=0.95 velocity=8.48 -> lower=-1.20 upper=1.90 effort=2.0 velocity=8.48
- joint leap_joint15: limit lower=-1.34 upper=1.88 effort=0.95 velocity=8.48 -> lower=-1.34 upper=1.88 effort=2.0 velocity=8.48
